Commit message: 小车仿真

File: adam_description/urdf/ackermann_mid360.urdf.xacro (robot description, xacro)
@@ -57,4 +57,10 @@
             </material>
         </visual>
+        <collision>
+            <origin xyz="0 0 0" rpy="1.57079 0 0"/>
+            <geometry>
+                <cylinder length="0.032" radius="0.04"/>
+            </geometry>
+        </collision>
         <xacro:cylinder_inertia m="0.5" r="0.04" h="0.032"/>
     </link>
@@ -64,4 +70,9 @@
         <origin xyz="0.08 0.07 -0.04" rpy="0 0 0"/>
     </joint>
+    <gazebo reference="front_left_wheel_link">
+        <material>Gazebo/Black</material>
+        <mu1>1.0</mu1>
+        <mu2>1.0</mu2>
+    </gazebo>
     <!-- 前右轮 -->
     <link name="front_right_wheel_link">
@@ -75,4 +86,10 @@
             </material>
         </visual>
+        <collision>
+            <origin xyz="0 0 0" rpy="1.57079 0 0"/>
+            <geometry>
+                <cylinder length="0.032" radius="0.04"/>
+            </geometry>
+        </collision>
         <xacro:cylinder_inertia m="0.5" r="0.04" h="0.032"/>
     </link>
@@ -82,4 +99,9 @@
         <origin xyz="0.08 -0.07 -0.04" rpy="0 0 0"/>
     </joint>
+    <gazebo reference="front_right_wheel_link">
+        <material>Gazebo/Black</material>
+        <mu1>1.0</mu1>
+        <mu2>1.0</mu2>
+    </gazebo>
     <!-- 后左轮 -->
     <link name="rear_left_wheel_link">
@@ -93,4 +115,10 @@
             </material>
         </visual>
+        <collision>
+            <origin xyz="0 0 0" rpy="1.57079 0 0"/>
+            <geometry>
+                <cylinder length="0.032" radius="0.04"/>
+            </geometry>
+        </collision>
         <xacro:cylinder_inertia m="0.5" r="0.04" h="0.032"/>
     </link>
@@ -100,4 +128,9 @@
         <origin xyz="-0.08 0.07 -0.04" rpy="0 0 0"/>
     </joint>
+    <gazebo reference="rear_left_wheel_link">
+        <material>Gazebo/Black</material>
+        <mu1>1.0</mu1>
+        <mu2>1.0</mu2>
+    </gazebo>
     <!-- 后右轮 -->
     <link name="rear_right_wheel_link">
@@ -111,4 +144,10 @@
             </material>
         </visual>
+        <collision>
+            <origin xyz="0 0 0" rpy="1.57079 0 0"/>
+            <geometry>
+                <cylinder length="0.032" radius="0.04"/>
+            </geometry>
+        </collision>
         <xacro:cylinder_inertia m="0.5" r="0.04" h="0.032"/>
     </link>
@@ -118,7 +157,12 @@
         <origin xyz="-0.08 -0.07 -0.04" rpy="0 0 0"/>
     </joint>
+    <gazebo reference="rear_right_wheel_link">
+        <material>Gazebo/Black</material>
+        <mu1>1.0</mu1>
+        <mu2>1.0</mu2>
+    </gazebo>
     <!-- =============== 传感器安装 =============== -->
-    <!-- Mid360 3D 激光雷达 (顶部中央) -->
-    <xacro:mid360 name="mid360" parent="base_link" topic="/livox/lidar">
+    <!-- 2D 激光雷达 (顶部中央) -->
+    <xacro:mid360 name="laser" parent="base_link">
         <origin xyz="0.0 0.0 0.06" rpy="0 0 0"/>
     </xacro:mid360>

File: adam_description/urdf/plugins/gazebo_sensors.xacro (robot description, xacro)
@@ -2,44 +2,7 @@
 <robot xmlns:xacro="http://www.ros.org/wiki/xacro">
     <!-- =============== Gazebo 传感器插件 =============== -->
-    <!-- 注意：IMU 传感器在各自的传感器 xacro 文件中定义 -->
+    <!-- 注意：传感器插件在各自的传感器 xacro 文件中定义 -->
+    <!-- 此文件保留用于未来扩展 -->
     <xacro:macro name="gazebo_sensors">
-        <!-- 2D 激光雷达 -->
-        <gazebo reference="laser_link">
-            <sensor name="laserscan" type="ray">
-                <plugin name="laser_plugin" filename="libgazebo_ros_ray_sensor.so">
-                    <ros>
-                        <namespace>/</namespace>
-                        <remapping>~/out:=scan</remapping>
-                    </ros>
-                    <output_type>sensor_msgs/LaserScan</output_type>
-                    <frame_name>laser_link</frame_name>
-                    <range_max>7.0</range_max>
-                </plugin>
-                <always_on>true</always_on>
-                <visualize>true</visualize>
-                <update_rate>10</update_rate>
-                <pose>0 0 0 0 0 0</pose>
-                <ray>
-                    <scan>
-                        <horizontal>
-                            <samples>360</samples>
-                            <resolution>1.0</resolution>
-                            <min_angle>0.0</min_angle>
-                            <max_angle>6.28</max_angle>
-                        </horizontal>
-                    </scan>
-                    <range>
-                        <min>0.12</min>
-                        <max>7.0</max>
-                        <resolution>0.015</resolution>
-                    </range>
-                    <noise>
-                        <type>gaussian</type>
-                        <mean>0.0</mean>
-                        <stddev>0.01</stddev>
-                    </noise>
-                </ray>
-            </sensor>
-        </gazebo>
     </xacro:macro>
 </robot>

File: adam_description/urdf/sensors/mid360.xacro (robot description, xacro)
@@ -25,14 +25,11 @@
         <origin xyz="0.025 -0.0265 -0.025" rpy="${pi/2} 0 ${pi}"/>
         <geometry>
-          <mesh filename="package://adam_description/data/meshes/mid360.stl" scale="0.0008 0.0008 0.0008"/>
+          <mesh filename="file://$(find adam_description)/data/meshes/mid360.stl" scale="0.0008 0.0008 0.0008"/>
         </geometry>
-        <material name="mid360_material">
-          <color rgba="0.2 0.2 0.2 1.0"/>
-        </material>
       </visual>
       <collision>
         <origin xyz="0.025 -0.0265 -0.025" rpy="${pi/2} 0 ${pi}"/>
         <geometry>
-          <mesh filename="package://adam_description/data/meshes/mid360.stl" scale="0.0008 0.0008 0.0008"/>
+          <mesh filename="file://$(find adam_description)/data/meshes/mid360.stl" scale="0.0008 0.0008 0.0008"/>
         </geometry>
       </collision>
