Commit message: fix center of mass

File: src/simulation/adam_description/urdf/ackermann_laser.urdf.xacro (robot description, xacro)
@@ -1,9 +1,9 @@
 <?xml version="1.0"?>
-<robot xmlns:xacro="http://www.ros.org/wiki/xacro" name="ackermann_mid360">
+<robot xmlns:xacro="http://www.ros.org/wiki/xacro" name="ackermann_laser">
     <!-- =============== 包含公共组件 =============== -->
     <xacro:include filename="$(find adam_description)/urdf/common/common_macros.xacro"/>
     <xacro:include filename="$(find adam_description)/urdf/common/common_inertia.xacro"/>
     <!-- =============== 包含传感器 =============== -->
-    <xacro:include filename="$(find adam_description)/urdf/sensors/mid360.xacro"/>
+    <xacro:include filename="$(find adam_description)/urdf/sensors/laser_2d.xacro"/>
     <xacro:include filename="$(find adam_description)/urdf/sensors/imu.xacro"/>
     <xacro:include filename="$(find adam_description)/urdf/sensors/mono_camera.xacro"/>
@@ -18,5 +18,5 @@
         <parent link="base_footprint"/>
         <child link="base_link"/>
-        <origin xyz="0 0 0.04" rpy="0 0 0"/>
+        <origin xyz="0 0 0.08" rpy="0 0 0"/>
     </joint>
     <link name="base_link">
@@ -163,7 +163,7 @@
     <!-- =============== 传感器安装 =============== -->
     <!-- 2D 激光雷达 (顶部中央) -->
-    <xacro:mid360 name="laser" parent="base_link">
+    <xacro:laser_2d name="laser" parent="base_link">
         <origin xyz="0.0 0.0 0.06" rpy="0 0 0"/>
-    </xacro:mid360>
+    </xacro:laser_2d>
     <!-- IMU (内部中央) -->
     <xacro:imu name="imu" parent="base_link">
@@ -174,5 +174,5 @@
         <origin xyz="0.12 0.0 0.03" rpy="0 0.2 0"/>
     </xacro:mono_camera>
-    <!-- 前向箭头（视觉指示） -->
+    <!-- 前向箭头（视觉指示）
     <link name="forward_arrow">
         <visual>
@@ -189,5 +189,5 @@
         <parent link="base_link"/>
         <child link="forward_arrow"/>
-    </joint>
+    </joint> -->
     <!-- =============== 应用插件 =============== -->
     <xacro:ros2_control/>

File: src/simulation/adam_description/urdf/ackermann_mid360.urdf.xacro (robot description, xacro)
@@ -1,9 +1,9 @@
 <?xml version="1.0"?>
-<robot xmlns:xacro="http://www.ros.org/wiki/xacro" name="ackermann_laser">
+<robot xmlns:xacro="http://www.ros.org/wiki/xacro" name="ackermann_mid360">
     <!-- =============== 包含公共组件 =============== -->
     <xacro:include filename="$(find adam_description)/urdf/common/common_macros.xacro"/>
     <xacro:include filename="$(find adam_description)/urdf/common/common_inertia.xacro"/>
     <!-- =============== 包含传感器 =============== -->
-    <xacro:include filename="$(find adam_description)/urdf/sensors/laser_2d.xacro"/>
+    <xacro:include filename="$(find adam_description)/urdf/sensors/mid360.xacro"/>
     <xacro:include filename="$(find adam_description)/urdf/sensors/imu.xacro"/>
     <xacro:include filename="$(find adam_description)/urdf/sensors/mono_camera.xacro"/>
@@ -18,5 +18,5 @@
         <parent link="base_footprint"/>
         <child link="base_link"/>
-        <origin xyz="0 0 0.04" rpy="0 0 0"/>
+        <origin xyz="0 0 0.08" rpy="0 0 0"/>
     </joint>
     <link name="base_link">
@@ -162,8 +162,8 @@
     </gazebo>
     <!-- =============== 传感器安装 =============== -->
-    <!-- 2D 激光雷达 (顶部中央) -->
-    <xacro:laser_2d name="laser" parent="base_link">
-        <origin xyz="0.0 0.0 0.06" rpy="0 0 0"/>
-    </xacro:laser_2d>
+    <!-- 3D 激光雷达 (顶部中央) -->
+    <xacro:mid360  name="livox_frame" parent="base_link" topic="/livox">
+        <origin xyz="0.0 0.0 0.06" rpy="0.0 0 0.0"/>
+    </xacro:mid360>
     <!-- IMU (内部中央) -->
     <xacro:imu name="imu" parent="base_link">
@@ -174,5 +174,5 @@
         <origin xyz="0.12 0.0 0.03" rpy="0 0.2 0"/>
     </xacro:mono_camera>
-    <!-- 前向箭头（视觉指示） -->
+    <!-- 前向箭头（视觉指示）
     <link name="forward_arrow">
         <visual>
@@ -189,5 +189,5 @@
         <parent link="base_link"/>
         <child link="forward_arrow"/>
-    </joint>
+    </joint> -->
     <!-- =============== 应用插件 =============== -->
     <xacro:ros2_control/>

File: src/simulation/adam_description/urdf/plugins/gazebo_control.xacro (robot description, xacro)
@@ -10,14 +10,14 @@
                     <namespace>/</namespace>
                     <remapping>cmd_vel:=/cmd_vel</remapping>
-                    <remapping>odom:=/odom</remapping>
+                    <remapping>odom:=/wheel_odom</remapping>
                 </ros>
                 <!-- 频率 -->
                 <update_rate>30</update_rate>
                 <!-- 里程计 frame id -->
-                <odometry_frame>odom</odometry_frame>
+                <odometry_frame>wheel_odom</odometry_frame>
                 <!-- 是否发布里程计 -->
                 <publish_odom>true</publish_odom>
                 <!-- 是否发布里程计 tf -->
-                <publish_odom_tf>true</publish_odom_tf>
+                <publish_odom_tf>false</publish_odom_tf>
                 <robot_base_frame>base_footprint</robot_base_frame>
                 <!-- 最大速度 -->

File: src/simulation/adam_description/urdf/sensors/mid360.xacro (robot description, xacro)
@@ -8,5 +8,5 @@
   <xacro:property name="noise_mean" value="0.0"/>
   <xacro:property name="noise_stddev" value="0.002"/>
-  <xacro:property name="mass" value="0.4" />
+  <xacro:property name="mass" value="0.1" /> <!-- 重心调不好 0.4 -> 0.1 -->
   <xacro:property name="length" value="0.1" />
   <xacro:property name="width" value="0.06" />
