Commit message: fix: 转弯翻车稳定性修复 — 加宽底盘/降低COM/降低摩擦/调小转弯加速度
稳定性修复：
- 加宽底盘 14cm→18cm，降低 COM 4cm→3cm，增大抗侧翻力矩
- 降低轮地摩擦 mu1/mu2=1.0→0.5，减少转弯侧向拖拽力
- 减小 max_vel_theta 1.0→0.6，max_accel_theta 0.5→0.3
- 加宽轮距 ±0.07→±0.085 匹配加宽底盘

Co-Authored-By: Claude Opus 4.7 <noreply@anthropic.com>

File: src/adam_description/urdf/ackermann_mid360.urdf.xacro (robot description, xacro)
@@ -15,9 +15,10 @@
     <!-- base_footprint 虚 link -->
     <link name="base_footprint"/>
-    <!-- base_link 主底盘 (长 240mm, 宽 140mm, 高 80mm) -->
+    <!-- base_link 主底盘 (长 240mm, 宽 180mm, 高 80mm) -->
     <joint name="base_joint" type="fixed">
         <parent link="base_footprint"/>
         <child link="base_link"/>
-        <origin xyz="0 0 0.04" rpy="0 0 0"/>
+        <!-- 降低 COM 高度以提高转弯稳定性 -->
+        <origin xyz="0 0 0.03" rpy="0 0 0"/>
     </joint>
     <link name="base_link">
@@ -25,5 +26,5 @@
             <origin xyz="0 0 0" rpy="0 0 0"/>
             <geometry>
-                <box size="0.24 0.14 0.08"/>
+                <box size="0.24 0.18 0.08"/>
             </geometry>
             <material name="base_material">
@@ -34,9 +35,9 @@
             <origin xyz="0 0 0" rpy="0 0 0"/>
             <geometry>
-                <box size="0.24 0.14 0.08"/>
+                <box size="0.24 0.18 0.08"/>
             </geometry>
             <material name="base_material"/>
         </collision>
-        <xacro:box_inertia m="1.5" w="0.24" h="0.08" d="0.14"/>
+        <xacro:box_inertia m="1.5" w="0.24" h="0.08" d="0.18"/>
     </link>
     <gazebo reference="base_link">
@@ -68,10 +69,10 @@
         <parent link="base_link"/>
         <child link="front_left_wheel_link"/>
-        <origin xyz="0.08 0.07 -0.04" rpy="0 0 0"/>
+        <origin xyz="0.08 0.085 -0.04" rpy="0 0 0"/>
     </joint>
     <gazebo reference="front_left_wheel_link">
         <material>Gazebo/Black</material>
-        <mu1>1.0</mu1>
-        <mu2>1.0</mu2>
+        <mu1>0.5</mu1>
+        <mu2>0.5</mu2>
     </gazebo>
     <!-- 前右轮 -->
@@ -97,10 +98,10 @@
         <parent link="base_link"/>
         <child link="front_right_wheel_link"/>
-        <origin xyz="0.08 -0.07 -0.04" rpy="0 0 0"/>
+        <origin xyz="0.08 -0.085 -0.04" rpy="0 0 0"/>
     </joint>
     <gazebo reference="front_right_wheel_link">
         <material>Gazebo/Black</material>
-        <mu1>1.0</mu1>
-        <mu2>1.0</mu2>
+        <mu1>0.5</mu1>
+        <mu2>0.5</mu2>
     </gazebo>
     <!-- 后左轮 -->
@@ -126,10 +127,10 @@
         <parent link="base_link"/>
         <child link="rear_left_wheel_link"/>
-        <origin xyz="-0.08 0.07 -0.04" rpy="0 0 0"/>
+        <origin xyz="-0.08 0.085 -0.04" rpy="0 0 0"/>
     </joint>
     <gazebo reference="rear_left_wheel_link">
         <material>Gazebo/Black</material>
-        <mu1>1.0</mu1>
-        <mu2>1.0</mu2>
+        <mu1>0.5</mu1>
+        <mu2>0.5</mu2>
     </gazebo>
     <!-- 后右轮 -->
@@ -155,10 +156,10 @@
         <parent link="base_link"/>
         <child link="rear_right_wheel_link"/>
-        <origin xyz="-0.08 -0.07 -0.04" rpy="0 0 0"/>
+        <origin xyz="-0.08 -0.085 -0.04" rpy="0 0 0"/>
     </joint>
     <gazebo reference="rear_right_wheel_link">
         <material>Gazebo/Black</material>
-        <mu1>1.0</mu1>
-        <mu2>1.0</mu2>
+        <mu1>0.5</mu1>
+        <mu2>0.5</mu2>
     </gazebo>
     <!-- =============== 传感器安装 =============== -->

File: src/adam_description/urdf/plugins/gazebo_control.xacro (robot description, xacro)
@@ -22,11 +22,11 @@
                 <robot_base_frame>base_footprint</robot_base_frame>
                 <!-- 最大速度 -->
-                <max_vel_x>1.0</max_vel_x>
+                <max_vel_x>0.8</max_vel_x>
                 <max_vel_y>0.0</max_vel_y>
-                <max_vel_theta>1.0</max_vel_theta>
+                <max_vel_theta>0.6</max_vel_theta>
                 <!-- 最大加速度 -->
-                <max_accel_x>0.5</max_accel_x>
+                <max_accel_x>0.4</max_accel_x>
                 <max_accel_y>0.0</max_accel_y>
-                <max_accel_theta>0.5</max_accel_theta>
+                <max_accel_theta>0.3</max_accel_theta>
             </plugin>
         </gazebo>

Commit message: fix: 修复转弯翻车 + 删除死代码 ros2_control
翻车根因:
- ros2_control.xacro 定义的关节不存在，导致 gazebo_ros2_control 加载失败
  并级联导致 planar_move 插件无法运行（报 parser error）
- 删除 ros2_control.xacro 引用后 planar_move 正常启动

URDF 修复:
- 底盘高度 base_joint: 0.03→0.09（底盘不再拖地）
- 轮子 joint origin: ±0.07/-0.04 → ±0.085/-0.05（轮底刚好接触地面）
- 底盘宽度: 0.14→0.18m（增大轮距）
- 轮地摩擦: mu1/mu2 1.0→0.5（减少侧向拖拽）
- max_vel_theta: 1.0→0.6, max_accel_theta: 0.5→0.3

验证: 持续右转 50 burst，z≈0，orientation x/y≈0，移动 2.66m 无翻车

Co-Authored-By: Claude Opus 4.7 <noreply@anthropic.com>

File: src/adam_description/urdf/ackermann_mid360.urdf.xacro (robot description, xacro)
@@ -9,5 +9,6 @@
     <xacro:include filename="$(find adam_description)/urdf/sensors/mono_camera.xacro"/>
     <!-- =============== 包含插件 =============== -->
-    <xacro:include filename="$(find adam_description)/urdf/plugins/ros2_control.xacro"/>
+    <!-- 注意: ros2_control.xacro 已注释掉 — URDF 中没有对应的 steering/drive 关节 -->
+    <!-- 机器人使用 planar_move 插件直接驱动底盘 -->
     <xacro:include filename="$(find adam_description)/urdf/plugins/gazebo_control.xacro"/>
     <xacro:include filename="$(find adam_description)/urdf/plugins/gazebo_sensors.xacro"/>
@@ -19,6 +20,6 @@
         <parent link="base_footprint"/>
         <child link="base_link"/>
-        <!-- 降低 COM 高度以提高转弯稳定性 -->
-        <origin xyz="0 0 0.03" rpy="0 0 0"/>
+        <!-- COM 高度: 轮子半径(0.04) + 底盘半高(0.04) + 间隙 → 0.09 -->
+        <origin xyz="0 0 0.09" rpy="0 0 0"/>
     </joint>
     <link name="base_link">
@@ -69,5 +70,5 @@
         <parent link="base_link"/>
         <child link="front_left_wheel_link"/>
-        <origin xyz="0.08 0.085 -0.04" rpy="0 0 0"/>
+        <origin xyz="0.08 0.085 -0.05" rpy="0 0 0"/>
     </joint>
     <gazebo reference="front_left_wheel_link">
@@ -98,5 +99,5 @@
         <parent link="base_link"/>
         <child link="front_right_wheel_link"/>
-        <origin xyz="0.08 -0.085 -0.04" rpy="0 0 0"/>
+        <origin xyz="0.08 -0.085 -0.05" rpy="0 0 0"/>
     </joint>
     <gazebo reference="front_right_wheel_link">
@@ -127,5 +128,5 @@
         <parent link="base_link"/>
         <child link="rear_left_wheel_link"/>
-        <origin xyz="-0.08 0.085 -0.04" rpy="0 0 0"/>
+        <origin xyz="-0.08 0.085 -0.05" rpy="0 0 0"/>
     </joint>
     <gazebo reference="rear_left_wheel_link">
@@ -156,5 +157,5 @@
         <parent link="base_link"/>
         <child link="rear_right_wheel_link"/>
-        <origin xyz="-0.08 -0.085 -0.04" rpy="0 0 0"/>
+        <origin xyz="-0.08 -0.085 -0.05" rpy="0 0 0"/>
     </joint>
     <gazebo reference="rear_right_wheel_link">
@@ -193,5 +194,4 @@
     </joint>
     <!-- =============== 应用插件 =============== -->
-    <xacro:ros2_control/>
     <xacro:gazebo_control/>
     <xacro:gazebo_sensors/>
