Commit message: feat: switch mid360 back to planar_move with anti-rollover optimization
- Changed all wheel joints from continuous to fixed (matching laser)
- Swapped plugin from gazebo_control_diff.xacro to gazebo_control.xacro
- Set wheel friction mu1/mu2=0.5 (was 0.8)
- Kept anti-rollover parameters: max_vel_theta=0.6, max_accel_theta=0.3
- Lowered COM height (base_joint z=0.03m)
- Updated documentation and cerebrum with proper simulation testing workflow

Testing: Three consecutive right-forward motion tests showed z≈0.06m, orientation x/y≈0 (no rollover)

File: src/adam_description/urdf/ackermann_mid360.urdf.xacro (robot description, xacro)
@@ -9,6 +9,6 @@
     <xacro:include filename="$(find adam_description)/urdf/sensors/mono_camera.xacro"/>
     <!-- =============== 包含插件 =============== -->
-    <!-- 使用 diff_drive 四轮差速控制（替代 planar_move 的 teleport 顿挫问题） -->
-    <xacro:include filename="$(find adam_description)/urdf/plugins/gazebo_control_diff.xacro"/>
+    <!-- 使用 planar_move 插件（丝滑运动） -->
+    <xacro:include filename="$(find adam_description)/urdf/plugins/gazebo_control.xacro"/>
     <xacro:include filename="$(find adam_description)/urdf/plugins/gazebo_sensors.xacro"/>
     <!-- =============== 创建机器人 =============== -->
@@ -19,6 +19,6 @@
         <parent link="base_footprint"/>
         <child link="base_link"/>
-        <!-- COM 高度: 轮子半径(0.04) + 底盘半高(0.04) + 间隙 → 0.09 -->
-        <origin xyz="0 0 0.09" rpy="0 0 0"/>
+        <!-- 降低 COM 高度以提高转弯稳定性: 0.09 → 0.03 -->
+        <origin xyz="0 0 0.03" rpy="0 0 0"/>
     </joint>
     <link name="base_link">
@@ -43,6 +43,6 @@
     <gazebo reference="base_link">
         <material>Gazebo/Blue</material>
-        <mu1>0.8</mu1>
-        <mu2>0.8</mu2>
+        <mu1>0.5</mu1>
+        <mu2>0.5</mu2>
     </gazebo>
     <!-- =============== 四轮驱动（四个 continuous joint） =============== -->
@@ -66,14 +66,13 @@
         <xacro:cylinder_inertia m="0.1" r="0.04" h="0.032"/>
     </link>
-    <joint name="front_left_wheel_joint" type="continuous">
+    <joint name="front_left_wheel_joint" type="fixed">
         <parent link="base_link"/>
         <child link="front_left_wheel_link"/>
         <origin xyz="0.08 0.085 -0.05" rpy="0 0 0"/>
-        <axis xyz="0 1 0"/>
     </joint>
     <gazebo reference="front_left_wheel_link">
         <material>Gazebo/Black</material>
-        <mu1>1.0</mu1>
-        <mu2>1.0</mu2>
+        <mu1>0.5</mu1>
+        <mu2>0.5</mu2>
     </gazebo>
     <!-- 前右轮 (continuous joint for driving) -->
@@ -96,14 +95,13 @@
         <xacro:cylinder_inertia m="0.1" r="0.04" h="0.032"/>
     </link>
-    <joint name="front_right_wheel_joint" type="continuous">
+    <joint name="front_right_wheel_joint" type="fixed">
         <parent link="base_link"/>
         <child link="front_right_wheel_link"/>
         <origin xyz="0.08 -0.085 -0.05" rpy="0 0 0"/>
-        <axis xyz="0 1 0"/>
     </joint>
     <gazebo reference="front_right_wheel_link">
         <material>Gazebo/Black</material>
-        <mu1>1.0</mu1>
-        <mu2>1.0</mu2>
+        <mu1>0.5</mu1>
+        <mu2>0.5</mu2>
     </gazebo>
     <!-- 后左轮 (continuous joint for driving) -->
@@ -126,14 +124,13 @@
         <xacro:cylinder_inertia m="0.1" r="0.04" h="0.032"/>
     </link>
-    <joint name="rear_left_wheel_joint" type="continuous">
+    <joint name="rear_left_wheel_joint" type="fixed">
         <parent link="base_link"/>
         <child link="rear_left_wheel_link"/>
         <origin xyz="-0.08 0.085 -0.05" rpy="0 0 0"/>
-        <axis xyz="0 1 0"/>
     </joint>
     <gazebo reference="rear_left_wheel_link">
         <material>Gazebo/Black</material>
-        <mu1>1.0</mu1>
-        <mu2>1.0</mu2>
+        <mu1>0.5</mu1>
+        <mu2>0.5</mu2>
     </gazebo>
     <!-- 后右轮 (continuous joint for driving) -->
@@ -156,14 +153,13 @@
         <xacro:cylinder_inertia m="0.1" r="0.04" h="0.032"/>
     </link>
-    <joint name="rear_right_wheel_joint" type="continuous">
+    <joint name="rear_right_wheel_joint" type="fixed">
         <parent link="base_link"/>
         <child link="rear_right_wheel_link"/>
         <origin xyz="-0.08 -0.085 -0.05" rpy="0 0 0"/>
-        <axis xyz="0 1 0"/>
     </joint>
     <gazebo reference="rear_right_wheel_link">
         <material>Gazebo/Black</material>
-        <mu1>1.0</mu1>
-        <mu2>1.0</mu2>
+        <mu1>0.5</mu1>
+        <mu2>0.5</mu2>
     </gazebo>
     <!-- =============== 传感器安装 =============== -->

File: src/adam_description/urdf/plugins/gazebo_control_diff.xacro (robot description, xacro)
@@ -13,4 +13,5 @@
                 <!-- 更新频率 -->
                 <update_rate>100</update_rate>
+                <publish_rate>10</publish_rate>
                 <!-- 里程计配置 -->
                 <odometry_frame>odom</odometry_frame>
@@ -18,15 +19,19 @@
                 <publish_odom>true</publish_odom>
                 <publish_odom_tf>true</publish_odom_tf>
-                <publish_wheel_tf>true</publish_wheel_tf>
-                <publishWheelJointState>true</publishWheelJointState>
+                <publish_wheel_tf>false</publish_wheel_tf>
+                <publishWheelJointState>false</publishWheelJointState>
+                <!-- 里程计协方差 -->
+                <covariance_x>0.0001</covariance_x>
+                <covariance_y>0.0001</covariance_y>
+                <covariance_yaw>0.01</covariance_yaw>
                 <!-- 后轮驱动，前轮 continuous 自由旋转（不拖拽） -->
                 <left_joint>rear_left_wheel_joint</left_joint>
                 <right_joint>rear_right_wheel_joint</right_joint>
-                <!-- 轮子几何 -->
-                <wheel_separation>0.18</wheel_separation>
+                <!-- 轮子几何 (与URDF实际轮距匹配: 0.085+0.085=0.17m) -->
+                <wheel_separation>0.17</wheel_separation>
                 <wheel_diameter>0.08</wheel_diameter>
-                <!-- 速度/扭矩限制：增大扭矩确保不打滑 -->
+                <!-- 速度/扭矩限制：增大扭矩和加速度确保充足驱动力和响应 -->
                 <max_wheel_torque>100</max_wheel_torque>
-                <max_wheel_acceleration>10.0</max_wheel_acceleration>
+                <max_wheel_acceleration>50.0</max_wheel_acceleration>
                 <command_topic>cmd_vel</command_topic>
                 <!-- 里程计源: 1=world (更平滑) -->
