Commit message: dev

File: src/adam_description/urdf/diff_drive_mid360.urdf.xacro (robot description, xacro)
@@ -1,4 +1,4 @@
 <?xml version="1.0"?>
-<robot xmlns:xacro="http://www.ros.org/wiki/xacro" name="ackermann_mid360">
+<robot xmlns:xacro="http://www.ros.org/wiki/xacro" name="diff_drive_mid360">
     <!-- =============== 包含公共组件 =============== -->
     <xacro:include filename="$(find adam_description)/urdf/common/common_macros.xacro"/>
@@ -9,5 +9,5 @@
     <xacro:include filename="$(find adam_description)/urdf/sensors/mono_camera.xacro"/>
     <!-- =============== 包含插件 =============== -->
-    <!-- 使用 diff_drive 四轮差速控制（替代 planar_move 的 teleport 顿挫问题） -->
+    <!-- diff_drive 四轮差速控制 -->
     <xacro:include filename="$(find adam_description)/urdf/plugins/gazebo_control_diff.xacro"/>
     <xacro:include filename="$(find adam_description)/urdf/plugins/gazebo_sensors.xacro"/>
@@ -46,6 +46,6 @@
         <mu2>0.8</mu2>
     </gazebo>
-    <!-- =============== 四轮驱动（四个 continuous joint） =============== -->
-    <!-- 前左轮 (continuous joint for driving) -->
+    <!-- =============== 四轮差速轮子 (continuous joints) =============== -->
+    <!-- 前左轮 -->
     <link name="front_left_wheel_link">
         <visual>
@@ -64,18 +64,17 @@
             </geometry>
         </collision>
-        <xacro:cylinder_inertia m="0.1" r="0.04" h="0.032"/>
+        <xacro:cylinder_inertia m="0.5" r="0.04" h="0.032"/>
     </link>
-    <joint name="front_left_wheel_joint" type="continuous">
+    <joint name="front_left_wheel_joint" type="fixed">
         <parent link="base_link"/>
         <child link="front_left_wheel_link"/>
         <origin xyz="0.08 0.085 -0.05" rpy="0 0 0"/>
-        <axis xyz="0 1 0"/>
     </joint>
     <gazebo reference="front_left_wheel_link">
         <material>Gazebo/Black</material>
-        <mu1>1.0</mu1>
-        <mu2>1.0</mu2>
+        <mu1>0.5</mu1>
+        <mu2>0.5</mu2>
     </gazebo>
-    <!-- 前右轮 (continuous joint for driving) -->
+    <!-- 前右轮 -->
     <link name="front_right_wheel_link">
         <visual>
@@ -94,18 +93,17 @@
             </geometry>
         </collision>
-        <xacro:cylinder_inertia m="0.1" r="0.04" h="0.032"/>
+        <xacro:cylinder_inertia m="0.5" r="0.04" h="0.032"/>
     </link>
-    <joint name="front_right_wheel_joint" type="continuous">
+    <joint name="front_right_wheel_joint" type="fixed">
         <parent link="base_link"/>
         <child link="front_right_wheel_link"/>
         <origin xyz="0.08 -0.085 -0.05" rpy="0 0 0"/>
-        <axis xyz="0 1 0"/>
     </joint>
     <gazebo reference="front_right_wheel_link">
         <material>Gazebo/Black</material>
-        <mu1>1.0</mu1>
-        <mu2>1.0</mu2>
+        <mu1>0.5</mu1>
+        <mu2>0.5</mu2>
     </gazebo>
-    <!-- 后左轮 (continuous joint for driving) -->
+    <!-- 后左轮 -->
     <link name="rear_left_wheel_link">
         <visual>
@@ -124,5 +122,5 @@
             </geometry>
         </collision>
-        <xacro:cylinder_inertia m="0.1" r="0.04" h="0.032"/>
+        <xacro:cylinder_inertia m="0.5" r="0.04" h="0.032"/>
     </link>
     <joint name="rear_left_wheel_joint" type="continuous">
@@ -134,8 +132,8 @@
     <gazebo reference="rear_left_wheel_link">
         <material>Gazebo/Black</material>
-        <mu1>1.0</mu1>
-        <mu2>1.0</mu2>
+        <mu1>0.5</mu1>
+        <mu2>0.5</mu2>
     </gazebo>
-    <!-- 后右轮 (continuous joint for driving) -->
+    <!-- 后右轮 -->
     <link name="rear_right_wheel_link">
         <visual>
@@ -154,5 +152,5 @@
             </geometry>
         </collision>
-        <xacro:cylinder_inertia m="0.1" r="0.04" h="0.032"/>
+        <xacro:cylinder_inertia m="0.5" r="0.04" h="0.032"/>
     </link>
     <joint name="rear_right_wheel_joint" type="continuous">
@@ -164,6 +162,6 @@
     <gazebo reference="rear_right_wheel_link">
         <material>Gazebo/Black</material>
-        <mu1>1.0</mu1>
-        <mu2>1.0</mu2>
+        <mu1>0.5</mu1>
+        <mu2>0.5</mu2>
     </gazebo>
     <!-- =============== 传感器安装 =============== -->

File: src/adam_description/urdf/sensors/mid360.xacro (robot description, xacro)
@@ -8,5 +8,5 @@
   <xacro:property name="noise_mean" value="0.0"/>
   <xacro:property name="noise_stddev" value="0.002"/>
-  <xacro:property name="mass" value="0.4" />
+  <xacro:property name="mass" value="0.15" />
   <xacro:property name="length" value="0.1" />
   <xacro:property name="width" value="0.06" />
