Commit message: feat: make simulation robot_description package independent by copying required data and worlds, finalize documentation

File: src/simulation/robot_description/urdf/sensors/mid360.xacro (robot description, xacro)
@@ -25,5 +25,5 @@
         <origin xyz="0.025 -0.0265 -0.025" rpy="${pi/2} 0 ${pi}"/>
         <geometry>
-          <mesh filename="file://$(find adam_description)/data/meshes/mid360.stl" scale="0.0008 0.0008 0.0008"/>
+          <mesh filename="file://$(find robot_description)/urdf/sensors/data/meshes/mid360.stl" scale="0.0008 0.0008 0.0008"/>
         </geometry>
       </visual>
@@ -31,5 +31,5 @@
         <origin xyz="0.025 -0.0265 -0.025" rpy="${pi/2} 0 ${pi}"/>
         <geometry>
-          <mesh filename="file://$(find adam_description)/data/meshes/mid360.stl" scale="0.0008 0.0008 0.0008"/>
+          <mesh filename="file://$(find robot_description)/urdf/sensors/data/meshes/mid360.stl" scale="0.0008 0.0008 0.0008"/>
         </geometry>
       </collision>
@@ -79,5 +79,5 @@
           <samples>${samples}</samples>
           <downsample>1</downsample>
-          <csv_file_name>$(find adam_description)/data/scan_mode/mid360.csv</csv_file_name>
+          <csv_file_name>$(find robot_description)/urdf/sensors/data/scan_mode/mid360.csv</csv_file_name>
           <topic>${topic}</topic>
         </plugin>
